Commit message: todo comentado y graficas con resultados

File: src/qr_robot_description/urdf/kobuki/kobuki.urdf.xacro (robot description, xacro)
@@ -265,5 +265,5 @@
   <joint name="camera_wide_joint" type="fixed">
     <axis xyz="0 1 0" />
-    <origin xyz="0.02 0 0.06" rpy="1.57 0 0"/>
+    <origin xyz="0.02 0 0.06" rpy="1.57 0 0"/> <!--1.57-->
     <parent link="camera_arm_02"/>
     <child link="camera_wide"/>
